Commit message: temp commit

File: dragon_ws/src/dragon_description/urdf/common.gazebo.xacro (robot description, xacro)
@@ -15,3 +15,19 @@
   	</plugin>
   </gazebo>
+    <!--color define-->
+  <gazebo reference="base_link">
+    <material>Gazebo/Green</material>
+  </gazebo>
+  <gazebo reference="leg_base">
+    <material>Gazebo/Turquoise</material>
+  </gazebo>
+  <gazebo reference="thigh">
+    <material>Gazebo/Blue</material>
+  </gazebo>
+  <gazebo reference="shank">
+    <material>Gazebo/Yellow</material>
+  </gazebo>
+  <gazebo reference="foot">
+    <material>Gazebo/Red</material>
+  </gazebo>
 </robot>

File: dragon_ws/src/dragon_description/urdf/single_leg.urdf.xacro (robot description, xacro)
@@ -10,17 +10,7 @@
     <child link="base_link" />
   </joint>
-  <link name="base_link">
-    <visual>
-      <geometry>
-        <sphere radius="0.0001"/>
-      </geometry>
-      <origin xyz="0 0 0" rpy="0 0 0" />
-    </visual>
-    <collision>
-      <geometry>
-        <sphere radius="0.0001"/>
-      </geometry>
-      <origin xyz="0 0 0" rpy="0 0 0" />
-    </collision>
+  <xacro:link_template name="base_link">
+    <sphere radius="0.0001"/>
+    <origin xyz="0 0 0" rpy="0 0 0" />
     <inertial>
       <origin xyz="0 0 0" rpy="0 0 0" />
@@ -28,7 +18,5 @@
       <inertia ixx="0" ixy="0.0" ixz="0.0" iyy="0" iyz="0.0" izz="0"/>
     </inertial>
-  </link>
-	<!-- single leg -->
-  <xacro:leg prefix=""/>
+  </xacro:link_template>
   <!-- The joint between the base of single leg and the world -->
   <joint name="base_link_to_base_joint" type="prismatic">
@@ -39,19 +27,15 @@
     <axis xyz="0 0 1" />
   </joint>
-  <!--color define-->
-  <gazebo reference="base_link">
-    <material>Gazebo/Green</material>
-  </gazebo>
-  <gazebo reference="leg_base">
-    <material>Gazebo/Turquoise</material>
-  </gazebo>
-  <gazebo reference="thigh">
-    <material>Gazebo/Blue</material>
-  </gazebo>
-  <gazebo reference="shank">
-    <material>Gazebo/Yellow</material>
-  </gazebo>
-  <gazebo reference="foot">
-    <material>Gazebo/Red</material>
-  </gazebo>
+  <!-- Only support obtain the joint state, The joint conn't be handled! -->
+  <transmission name="base_link_to_base_joint_trans">
+    <type>transmission_interface/SimpleTransmission</type>
+    <joint name="base_link_to_base_joint">
+      <hardwareInterface>EffortJointInterface</hardwareInterface>
+    </joint>
+    <actuator name="base_link_to_base_joint_motor">
+      <mechanicalReduction>0</mechanicalReduction>
+    </actuator>
+  </transmission>
+	<!-- single leg -->
+  <xacro:leg prefix=""/>
 </robot>

Commit message: model y-z

File: dragon_ws/src/dragon_description/urdf/common.gazebo.xacro (robot description, xacro)
@@ -9,5 +9,5 @@
       <!--robotNamespace>your_robot_name</robotNamespace-->
       <jointName>
-          base_link_to_base_joint, hip, knee
+          hip, knee
       </jointName>
       <updateRate>100</updateRate>

File: dragon_ws/src/dragon_description/urdf/leg.urdf.xacro (robot description, xacro)
@@ -75,5 +75,4 @@
 	    <origin xyz="0 0 0" rpy="0 0 0"/>
 	    <dynamics damping="0" friction="0"/>
-	    <!--limit lower="-0.78539815" upper="0.698131689" effort="100" velocity="100"/-->
 	    <limit lower="${-0.4*pi/2}" upper="${-0.01*pi/2}" effort="100" velocity="100"/>
 	  </joint>

File: dragon_ws/src/dragon_description/urdf/single_leg.urdf.xacro (robot description, xacro)
@@ -5,10 +5,5 @@
   <!-- single leg XACRO -->
   <xacro:include filename="$(find dragon_description)/urdf/leg.urdf.xacro" />
-  <link name="world" />
-  <joint name="world_to_base_link_joint" type="fixed" >
-    <parent link="world" />
-    <child link="base_link" />
-  </joint>
-  <xacro:link_template name="base_link">
+  <!--xacro:link_template name="base_link">
     <sphere radius="0.0001"/>
     <origin xyz="0 0 0" rpy="0 0 0" />
@@ -18,24 +13,60 @@
       <inertia ixx="0" ixy="0.0" ixz="0.0" iyy="0" iyz="0.0" izz="0"/>
     </inertial>
-  </xacro:link_template>
-  <!-- The joint between the base of single leg and the world -->
-  <joint name="base_link_to_base_joint" type="prismatic">
-    <parent link="base_link" />
-    <child link = "leg_base" />
-    <origin xyz="0.0 0.0 0.0" rpy="0.0 0.0 0.0" />
-    <limit lower="-0.1" upper="2.0" effort="100" velocity="100"/>
+  </xacro:link_template-->
+  <link name="world" />
+  <joint name="y_axis_joint" type="fixed">
+    <parent link="world" />
+    <child link="framework" />
+    <origin xyz="0.0 0.0 0" rpy="0.0 0.0 0.0" />
+  </joint>
+  <xacro:link_stl_template name="framework" stl="main1n">
+    <origin xyz="0 0 0" rpy="0 0 0" />
+    <inertial>
+      <origin xyz="0 0 0" rpy="0 0 0"/>
+      <mass value="10" />
+      <inertia ixx="0" ixy="0" ixz="0" iyy="0" iyz="0" izz="0"/>
+    </inertial>
+  </xacro:link_stl_template>
+  <!--xacro:link_template name="y_axis">
+    <box size="0.01 0.02 5"/>
+    <origin xyz="0 -0.04 0" rpy="0 ${pi/2} 0" />
+    <inertial>
+      <origin xyz="0 0 0" rpy="0 0 0" />
+      <mass value="0"/>
+      <inertia ixx="0" ixy="0.0" ixz="0.0" iyy="0" iyz="0.0" izz="0"/>
+    </inertial>
+  </xacro:link_template-->
+  <joint name="z_axis_joint" type="prismatic">
+    <parent link="framework" />
+    <child link="z_axis" />
+    <origin xyz="0.0 0.0 0.2" rpy="0.0 0.0 0.0" />
+    <limit lower="-0.9" upper="0.9" effort="100" velocity="10"/>
+    <axis xyz="1 0 0" />
+  </joint>
+  <xacro:link_stl_template name="z_axis" stl="main2n">
+    <origin xyz="0 0 0" rpy="0 0 0" />
+    <inertial>
+      <origin xyz="0 0 0" rpy="0 0 0"/>
+      <mass value="0.0001" />
+      <inertia ixx="0" ixy="0" ixz="0" iyy="0" iyz="0" izz="0"/>
+    </inertial>
+  </xacro:link_stl_template>
+  <!--xacro:link_template name="z_axis">
+    <box size="0.01 0.02 3"/>
+    <origin xyz="0.1 -0.03 1.2" rpy="0 0 ${pi/2}" />
+    <inertial>
+      <origin xyz="0 0 0" rpy="0 0 0" />
+      <mass value="0.0001"/>
+      <inertia ixx="0" ixy="0.0" ixz="0.0" iyy="0" iyz="0.0" izz="0"/>
+    </inertial>
+  </xacro:link_template-->
+  <joint name="axis_to_base_joint" type="prismatic">
+    <parent link="z_axis" />
+    <child link="leg_base" />
+    <origin xyz="0 0.06 0.5" rpy="0.0 0.0 0.0" />
+    <limit lower="-0.2" upper="0.4" effort="100" velocity="10"/>
     <axis xyz="0 0 1" />
   </joint>
-  <!-- Only support obtain the joint state, The joint conn't be handled! -->
-  <transmission name="base_link_to_base_joint_trans">
-    <type>transmission_interface/SimpleTransmission</type>
-    <joint name="base_link_to_base_joint">
-      <hardwareInterface>EffortJointInterface</hardwareInterface>
-    </joint>
-    <actuator name="base_link_to_base_joint_motor">
-      <mechanicalReduction>0</mechanicalReduction>
-    </actuator>
-  </transmission>
-	<!-- single leg -->
+  <!-- single leg -->
   <xacro:leg prefix=""/>
 </robot>

Commit message: tmp

File: dragon_ws/src/dragon_description/urdf/common.gazebo.xacro (robot description, xacro)
@@ -9,5 +9,5 @@
       <!--robotNamespace>your_robot_name</robotNamespace-->
       <jointName>
-          hip, knee
+          z_axis_joint, axis_to_base_joint, hip, knee
       </jointName>
       <updateRate>100</updateRate>

File: dragon_ws/src/dragon_description/urdf/leg.urdf.xacro (robot description, xacro)
@@ -1,4 +1,6 @@
 <?xml version="1.0" ?>
 <robot xmlns:xacro="http://www.ros.org/wiki/xacro">
+	<property name="effort" value="30.0" />
+  <property name="velocity" value="5.0" />
 	<!-- define transmission -->
   <xacro:include filename="$(find dragon_description)/urdf/leg.transmission.xacro" />
@@ -75,5 +77,5 @@
 	    <origin xyz="0 0 0" rpy="0 0 0"/>
 	    <dynamics damping="0" friction="0"/>
-	    <limit lower="${-0.4*pi/2}" upper="${-0.01*pi/2}" effort="100" velocity="100"/>
+	    <limit lower="${-0.4*pi/2}" upper="${-0.01*pi/2}" effort="${effort}" velocity="${velocity}"/>
 	  </joint>
 	  <xacro:link_stl_template name="${prefix}thigh" stl="upper_leg">
@@ -92,5 +94,5 @@
 	    <dynamics damping="0" friction="0"/>
 	    <!--limit lower="0.174532922" upper="1.919862144" effort="100" velocity="100"/-->
-	    <limit lower="${-0.01*pi/2}" upper="${0.6*pi/2}" effort="100" velocity="100"/>
+	    <limit lower="${-0.01*pi/2}" upper="${0.6*pi/2}" effort="${effort}" velocity="${velocity}"/>
 	  </joint>
 	  <xacro:link_stl_template name="${prefix}shank" stl="back_shine">

File: dragon_ws/src/dragon_description/urdf/single_leg.urdf.xacro (robot description, xacro)
@@ -41,5 +41,5 @@
     <child link="z_axis" />
     <origin xyz="0.0 0.0 0.2" rpy="0.0 0.0 0.0" />
-    <limit lower="-0.9" upper="0.9" effort="100" velocity="10"/>
+    <limit lower="-0.9" upper="0.9" effort="${effort}" velocity="${velocity}"/>
     <axis xyz="1 0 0" />
   </joint>
@@ -65,8 +65,28 @@
     <child link="leg_base" />
     <origin xyz="0 0.06 0.5" rpy="0.0 0.0 0.0" />
-    <limit lower="-0.2" upper="0.4" effort="100" velocity="10"/>
+    <limit lower="-0.45" upper="0.4" effort="${effort}" velocity="${velocity}"/>
     <axis xyz="0 0 1" />
   </joint>
+  <!-- Only support obtain the joint state, The joint conn't be handled! -->
+  <transmission name="z_axis_joint_trans">
+    <type>transmission_interface/SimpleTransmission</type>
+    <joint name="z_axis_joint">
+      <hardwareInterface>EffortJointInterface</hardwareInterface>
+    </joint>
+    <actuator name="z_axis_joint_motor">
+      <mechanicalReduction>0</mechanicalReduction>
+    </actuator>
+  </transmission>
+  <!-- Only support obtain the joint state, The joint conn't be handled! -->
+  <transmission name="axis_to_base_joint_trans">
+    <type>transmission_interface/SimpleTransmission</type>
+    <joint name="axis_to_base_joint">
+      <hardwareInterface>EffortJointInterface</hardwareInterface>
+    </joint>
+    <actuator name="axis_to_base_joint_motor">
+      <mechanicalReduction>0</mechanicalReduction>
+    </actuator>
+  </transmission>
   <!-- single leg -->
-  <xacro:leg prefix=""/>
+  <xacro:leg prefix="" />
 </robot>
