Commit message: model color set by wang

File: dragon_ws/src/dragon_description/urdf/single_leg.urdf.xacro (robot description, xacro)
@@ -39,3 +39,19 @@
     <axis xyz="0 0 1" />
   </joint>
+  <!--color define-->
+  <gazebo reference="base_link">
+    <material>Gazebo/Green</material>
+  </gazebo>
+  <gazebo reference="leg_base">
+    <material>Gazebo/Turquoise</material>
+  </gazebo>
+  <gazebo reference="thigh">
+    <material>Gazebo/Blue</material>
+  </gazebo>
+  <gazebo reference="shank">
+    <material>Gazebo/Yellow</material>
+  </gazebo>
+  <gazebo reference="foot">
+    <material>Gazebo/Red</material>
+  </gazebo>
 </robot>

Commit message: completed the single leg hopping in only one DoF(z axis)

File: dragon_ws/src/dragon_description/urdf/single_leg.urdf.xacro (robot description, xacro)
@@ -23,6 +23,6 @@
     <parent link="base_link" />
     <child link = "leg_base" />
-    <origin xyz="0.0 0.0 0.7" rpy="0.0 0.0 0.0" />
-    <limit lower="-0.7" upper="1.0" effort="100" velocity="100"/>
+    <origin xyz="0.0 0.0 0.0" rpy="0.0 0.0 0.0" />
+    <limit lower="-0.1" upper="2.0" effort="100" velocity="100"/>
     <axis xyz="0 0 1" />
   </joint>

Commit message: trans del

File: dragon_ws/src/dragon_description/urdf/single_leg.urdf.xacro (robot description, xacro)
@@ -40,5 +40,5 @@
     <parent link="framework" />
     <child link="z_axis" />
-    <origin xyz="0.0 0.0 0.2" rpy="0.0 0.0 0.0" />
+    <origin xyz="0.0 -0.035 0.2" rpy="0.0 0.0 0.0" />
     <limit lower="-0.9" upper="0.9" effort="${effort}" velocity="${velocity}"/>
     <axis xyz="1 0 0" />
@@ -64,10 +64,10 @@
     <parent link="z_axis" />
     <child link="leg_base" />
-    <origin xyz="0 0.06 0.5" rpy="0.0 0.0 0.0" />
+    <origin xyz="-0.1 0.06 0.5" rpy="0.0 0.0 0.0" />
     <limit lower="-0.45" upper="0.4" effort="${effort}" velocity="${velocity}"/>
     <axis xyz="0 0 1" />
   </joint>
   <!-- Only support obtain the joint state, The joint conn't be handled! -->
-  <transmission name="z_axis_joint_trans">
+  <!--transmission name="z_axis_joint_trans">
     <type>transmission_interface/SimpleTransmission</type>
     <joint name="z_axis_joint">
@@ -77,7 +77,7 @@
       <mechanicalReduction>0</mechanicalReduction>
     </actuator>
-  </transmission>
+  </transmission-->
   <!-- Only support obtain the joint state, The joint conn't be handled! -->
-  <transmission name="axis_to_base_joint_trans">
+  <!--transmission name="axis_to_base_joint_trans">
     <type>transmission_interface/SimpleTransmission</type>
     <joint name="axis_to_base_joint">
@@ -87,5 +87,5 @@
       <mechanicalReduction>0</mechanicalReduction>
     </actuator>
-  </transmission>
+  </transmission-->
   <!-- single leg -->
   <xacro:leg prefix="" />
